Commit message: wip: backup in-progress work after power outage
Snapshot of uncommitted changes interrupted by power loss during training.
Includes:
- new stand-in-place task cfg (LeRobotStandEnvCfg) and velocity env tweaks
- actuator / observation / reward / termination adjustments
- PPO + actor-critic tweaks
- hot_diagnosis additions: alpha1_check.py, summary_metrics.py, plus
  updates to diagnose / fetch / go_to_zero / onnx_replay / sim_rollout
- export_onnx and sim2mujoco_watcher fixes

Co-Authored-By: Claude Opus 4.7 (1M context) <noreply@anthropic.com>
Signed-off-by: haixuantao <tao.xavier@outlook.com>

File: agile/rl_env/assets/robots/lerobot_humanoid_no_arms_new.urdf (robot description, URDF)
Before this commit: robot lerobot_humanoid_no_arms, 16 links, 15 joints
Joints:
- joint hipx_left: limit lower=-0.349066 upper=0.349066 effort=10 velocity=10 -> lower=-0.5342 upper=1.2112 effort=10 velocity=10
- joint hipx_right: limit lower=-0.349066 upper=0.349066 effort=10 velocity=10 -> lower=-1.2112 upper=0.5342 effort=10 velocity=10
- joint hipy_left: limit lower=-1.0472 upper=1.0472 effort=10 velocity=10 -> lower=-1.3957 upper=1.5376 effort=10 velocity=10
- joint hipy_right: limit lower=-1.0472 upper=1.0472 effort=10 velocity=10 -> lower=-1.5376 upper=1.2975 effort=10 velocity=10
- joint hipz_left: limit lower=-0.349066 upper=0.349066 effort=10 velocity=10 -> lower=-1.3495 upper=1.4430 effort=10 velocity=10
- joint hipz_right: limit lower=-0.349066 upper=0.349066 effort=10 velocity=10 -> lower=-1.4430 upper=1.3495 effort=10 velocity=10
- joint knee_left: limit lower=-0.523599 upper=0.523599 effort=10 velocity=10 -> lower=-0.9568 upper=0.9839 effort=10 velocity=10
- joint knee_right: limit lower=-0.523599 upper=0.523599 effort=10 velocity=10 -> lower=-0.7113 upper=0.9889 effort=10 velocity=10
